Commit message: Actualizar stl

File: limo_description/urdf/limo_xacro.xacro (robot description, xacro)
@@ -15,15 +15,15 @@
             </visual>
             <collision>
-                <origin xyz="0 ${wheel_length/2} 0" rpy="1.57 0 0" />
-                <geometry>
-                    <cylinder length="${wheel_length}" radius="${wheel_radius}" />
-                </geometry>
+              <origin xyz="0 ${wheel_length/2} 0" rpy="1.57 0 0" />
+              <geometry>
+                  <cylinder length="${wheel_length}" radius="${wheel_radius}" />
+              </geometry>
             </collision>
         </link>
         <joint name="${wheel_prefix}_wheel" type="continuous">
-            <parent link="${parent_prefix}" />
-            <child link="${wheel_prefix}_wheel_link" />
-            <xacro:insert_block name="joint_pose" />
-            <axis xyz="0 ${reflect*1} 0" />
+            <parent link="${parent_prefix}"/>
+            <child link="${wheel_prefix}_wheel_link"/>
+            <xacro:insert_block name="joint_pose"/>
+            <axis xyz="0 ${reflect*1} 0"/>
         </joint>
     </xacro:macro>
@@ -31,7 +31,7 @@
         <link name='${frame_prefix}_link' />
         <joint type="fixed" name="laser_joint">
-            <xacro:insert_block name="joint_pose" />
-            <child link="${frame_prefix}_link" />
-            <parent link="${parent_prefix}" />
+            <xacro:insert_block name="joint_pose"/>
+            <child link="${frame_prefix}_link"/>
+            <parent link="${parent_prefix}"/>
         </joint>
     </xacro:macro>
@@ -39,28 +39,23 @@
         <link name='${frame_prefix}_link' />
         <joint type="fixed" name="depth_camera_joint">
-            <xacro:insert_block name="joint_pose" />
-            <child link="${frame_prefix}_link" />
-            <parent link="${parent_prefix}" />
+            <xacro:insert_block name="joint_pose"/>
+            <child link="${frame_prefix}_link"/>
+            <parent link="${parent_prefix}"/>
         </joint>
         <link name="depth_link" />
         <joint name="${frame_prefix}_to_camera_joint" type="fixed">
-            <origin xyz="0 0 0" rpy="${-M_PI/2} 0 ${-M_PI/2} " />
-            <parent link="${frame_prefix}_link" />
-            <child link="depth_link" />
+            <origin xyz="0 0 0" rpy="${-M_PI/2} 0 ${-M_PI/2} "/>
+            <parent link="${frame_prefix}_link"/>
+            <child link="depth_link"/>
+          </joint>
+    </xacro:macro>
+    <xacro:macro name="limo_imu" params="parent_prefix frame_prefix  *joint_pose">
+        <link name='${frame_prefix}_link'/>
+        <joint type="fixed" name="imu_joint">
+            <xacro:insert_block name="joint_pose"/>
+            <child link="${frame_prefix}_link"/>
+            <parent link="${parent_prefix}"/>
         </joint>
     </xacro:macro>
-    <xacro:macro name="limo_imu" params="parent_prefix frame_prefix  *joint_pose">
-        <link name='${frame_prefix}_link' />
-        <joint type="fixed" name="imu_joint">
-            <xacro:insert_block name="joint_pose" />
-            <child link="${frame_prefix}_link" />
-            <parent link="${parent_prefix}" />
-        </joint>
-    </xacro:macro>
-    <gazebo reference="${wheel_prefix}_wheel_link">
-        <mu1>0.5</mu1>   <!-- Coeficiente de fricción longitudinal -->
-        <mu2>0.5</mu2>   <!-- Coeficiente de fricción lateral -->
-        <kp>1000.0</kp>  <!-- Incrementa el factor de rigidez -->
-        <kd>10.0</kd>    <!-- Ajusta el amortiguamiento -->
-    </gazebo>
+    <xacro:include filename="$(optenv URDF_EXTENSION empty.urdf)" />
 </robot>
